File: FilPilote/FilPilote.kicad_pcb (KiCad board)
At the start: 2 copper layers, 23 parts, among them J1 Conn_01x04_Male, P1 CONN_01X03, Q1 AO3400, Q2 AO3400, SW1 RESET, SW2 FLASH, U1 MOC3041M, U2 MOC3041M, U3 AMS1117, U4 ESP-12E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

Commit message: Finished FilPilote schematic + PCB
Parts:
- removed C1: 10u, Capacitor_SMD:C_1206_3216Metric_Pad1.42x1.75mm_HandSolder
- removed Q1, Q2: AO3400, Package_TO_SOT_SMD:SOT-23
- removed R3, R5: 100, Resistor_SMD:R_0805_2012Metric_Pad1.15x1.40mm_HandSolder
- removed R4, R6: 1M, Resistor_SMD:R_0805_2012Metric_Pad1.15x1.40mm_HandSolder
- removed U3: AMS1117, Package_TO_SOT_SMD:SOT-223-3_TabPin2
- C3: value 10u -> 100nF; moved to B.Cu
- D1, D2: footprint Diode_THT:D_DO-41_SOD81_P7.62mm_Horizontal -> Diode_SMD:D_SOD-123
- R1, R2: value 300 -> 270
- R7, R8: moved to B.Cu
- U5: value HLK-PM01 -> HLK-PM03
- moved FLASH 32.3 mm to (158.0, 87.2)
- moved J1 31.4 mm to (133.9, 101.2), turned to 0 degrees
- moved RST 18.3 mm to (158.0, 77.2), turned to 90 degrees
- moved R8 8.37 mm to (142.1, 103.1), turned to 180 degrees
- moved U4 7.22 mm to (149.1, 102.3)
- moved D1 4.41 mm to (127.0, 95.0)
- moved R7 4.07 mm to (149.6, 98.8)
- moved R2 3.10 mm to (114.7, 108.7)
- moved R1 2.75 mm to (124.6, 108.7), turned to 0 degrees
- moved U2 2.57 mm to (113.9, 105.8)
- moved U1 2.45 mm to (123.6, 105.7)
- moved C3 2.38 mm to (142.5, 98.9)
- moved D2 1.94 mm to (117.3, 95.1)
- renumbered SW2 to FLASH, SW1 to RST
Connections:
- C3 pad 1: /3V3 -> /GND
- C3 pad 2: /GND -> /3V3
- R1 pad 2: /3V3 -> /O1
- R2 pad 2: /3V3 -> /O2
- U1 pad 2: /O1 -> /GND
- U2 pad 2: /O2 -> /GND
- U4 pad 6: /S_OP1 -> /O1
- U4 pad 7: /S_OP2 -> /O2
- U5 pad 4: /VCC -> /3V3
Routing:
- net /PH_IN: track 0.00 -> 45.3 mm
- net /3V3: track 0.00 -> 42.8 mm, vias 0 -> 1
- net /O2: track 0.00 -> 40.2 mm
- net Net-(R8-Pad1): track 0.00 -> 39.7 mm, vias 0 -> 2
- net /O1: track 0.00 -> 31.7 mm
- net Net-(R7-Pad1): track 0.00 -> 29.6 mm, vias 0 -> 1
- net /TXD: track 0.00 -> 22.6 mm, vias 0 -> 1
- net /RXD: track 0.00 -> 19.8 mm, vias 0 -> 1
- net /FP_OUT: track 0.00 -> 17.6 mm
- net /NEUTRE: track 0.00 -> 7.08 mm
- net Net-(D1-Pad2): track 0.00 -> 3.05 mm
- net Net-(D2-Pad1): track 0.00 -> 3.05 mm
- net Net-(R2-Pad1): track 0.00 -> 3.03 mm
- net Net-(R1-Pad1): track 0.00 -> 2.79 mm
- added copper zone on B.Cu, net /GND
- added copper zone on F.Cu, net /GND
Other:
- board outline added: 50 x 40 mm
